Commit message: Created a depth visualisation

File: legged_gym/resources/robots/wf_tron1a/urdf/robot.urdf (robot description, URDF)
Before this commit: robot wheel_biped, 10 links, 9 joints
Links:
- added link d435_Link; collision box size=0.02505 0.09 0.025; visual box size=0.02505 0.09 0.025
Joints:
- added joint d435_joint: type fixed, parent base_Link, child d435_Link, origin xyz=0.13223 0.0222 -0.26826 rpy=0 1.063778179 0
